File: Arduino/Uno/Uno_RF24.kicad_pcb (KiCad board)
At the start: 2 copper layers, 68.8 x 53.6 mm, 4 parts, among them P1 Remove jumpers if using ICSP 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, P2 NRF24L01+, U1 NRF24L01+ Shield

Commit message: Update URLs and images
Other:
- board text added: "github.com/markjb/NRF24L01_Adaptors"
- board text removed: "github.com/markjb/url?"
Changed lines of the file:
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@@
     (comment 1 "Copyright Mark Benson 2016")
     (comment 2 "License: Creative Commons Attribution Non Commercial (CCNCBY 4.0)")
-    (comment 3 github.com/markjb/url)
+    (comment 3 github.com/markjb/NRF24L01_Adaptors)
   )
   (layers
@@
   (gr_circle (center 174.752 60.452) (end 174.752 60.706) (layer F.SilkS) (width 0.2))
   (gr_circle (center 174.752 59.436) (end 174.752 59.69) (layer F.SilkS) (width 0.2))
-  (gr_text github.com/markjb/url? (at 159.512 83.82) (layer F.SilkS)
+  (gr_text github.com/markjb/NRF24L01_Adaptors (at 165.608 83.82) (layer F.SilkS)
     (effects (font (size 1 1) (thickness 0.15)))
   )
