File: Raspberry_Pi/rasberry_pi_minimal_rf24_board.kicad_pcb (KiCad board)
At the start: 2 copper layers, 52.8 x 24.3 mm, 3 parts, among them P1 RPi, P2 NRF24L01+

Commit message: Update URLs and images
Other:
- board text added: "github.com/markjb/NRF24L01_Adaptors"
- board text removed: "github.com/markjb/url?"
Changed lines of the file:
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@@
     (comment 1 "Copyright Mark Benson 2016")
     (comment 2 "License: Creative Commons Attribution Non Commerical 4.0 (CCNCBY 4.0)")
-    (comment 3 github.com/markjb/url)
+    (comment 3 github.com/markjb/NRF24L01_Adaptors)
   )
   (layers
@@
   (gr_line (start 126.5936 88.6968) (end 177.4444 88.6968) (angle 90) (layer Edge.Cuts) (width 0.15))
   (gr_line (start 177.4952 95.504) (end 174.1424 95.504) (angle 90) (layer Edge.Cuts) (width 0.15))
-  (gr_text github.com/markjb/url? (at 153.924 100.33) (layer F.SilkS)
-    (effects (font (size 1 1) (thickness 0.15)))
+  (gr_text github.com/markjb/NRF24L01_Adaptors (at 156.972 100.33) (layer F.SilkS)
+    (effects (font (size 0.8 0.8) (thickness 0.15)))
   )
   (gr_text "©Mark Benson 2016 CCNCBY4.0" (at 157.226 98.298) (layer F.SilkS)
@@
   (gr_arc (start 126.5428 89.6112) (end 125.6284 89.5604) (angle 90) (layer Edge.Cuts) (width 0.15))
   (gr_arc (start 177.4952 89.6112) (end 177.4444 88.6968) (angle 90) (layer Edge.Cuts) (width 0.15))
-  (segment (start 159.2961 110.8456) (end 160.6677 109.474) (width 0.25) (layer B.Cu) (net 1) (status 400000))
-  (segment (start 167.386 107.95) (end 167.386 105.41) (width 0.25) (layer B.Cu) (net 1) (status 800000))
+  (segment (start 159.2961 110.8456) (end 160.6677 109.474) (width 0.25) (layer B.Cu) (net 1))
+  (segment (start 167.386 107.95) (end 167.386 105.41) (width 0.25) (layer B.Cu) (net 1))
   (segment (start 165.862 109.474) (end 167.386 107.95) (width 0.25) (layer B.Cu) (net 1))
   (segment (start 160.6677 109.474) (end 165.862 109.474) (width 0.25) (layer B.Cu) (net 1))
@@
   (segment (start 148.336 105.8672) (end 148.336 93.4212) (width 0.25) (layer B.Cu) (net 1))
   (segment (start 153.3144 110.8456) (end 148.336 105.8672) (width 0.25) (layer B.Cu) (net 1))
-  (segment (start 161.8361 110.8456) (end 166.7764 110.8456) (width 0.25) (layer F.Cu) (net 2) (status 400000))
-  (segment (start 169.386 108.236) (end 169.386 105.41) (width 0.25) (layer F.Cu) (net 2) (status 800000))
+  (segment (start 161.8361 110.8456) (end 166.7764 110.8456) (width 0.25) (layer F.Cu) (net 2))
+  (segment (start 169.386 108.236) (end 169.386 105.41) (width 0.25) (layer F.Cu) (net 2))
   (segment (start 166.7764 110.8456) (end 169.386 108.236) (width 0.25) (layer F.Cu) (net 2))
   (segment (start 161.8361 110.8456) (end 160.5153 112.1664) (width 0.25) (layer F.Cu) (net 2))
